File: modular_device_base_3x2.kicad_pcb (KiCad board)
At the start: 2 copper layers, 83.8 x 40.6 mm, 23 parts, among them P1 PWR_JACK_2.5x5.5_SMD_RA, P2 HEADER_01X03_SMD_RA, P3 HEADER_01X03_SMD_RA, P4 HEADER_01X03_SMD_RA, P5 BNC_DOUBLE_RA, P6 HEADER_01X02_SMD_RA, P7 HEADER_01X02_SMD_RA, SW1 KT_SWITCH

Commit message: modular_device_teensy -> modular_device_base.
Parts:
- C1, C2, C3, C4, C5: footprint modular_device_teensy_3x2:SM1210 -> modular_device_base_3x2:SM1210
- D1, D2: footprint modular_device_teensy_3x2:DO-214BA -> modular_device_base_3x2:DO-214BA
- D3, D4: footprint modular_device_teensy_3x2:CFP15 -> modular_device_base_3x2:CFP15
- MDT1: value MODULAR_DEVICE_TEENSY_3X2_FEMALE -> MODULAR_DEVICE_BASE_3X2_FEMALE; footprint modular_device_teensy_3x2:MODULAR_DEVICE_TEENSY_3X2_FEMALE -> modular_device_base_3x2:MODULAR_DEVICE_BASE_3X2_FEMALE
- MH1, MH2, MH3: footprint modular_device_teensy_3x2:MOUNTING_HOLE_4-40 -> modular_device_base_3x2:MOUNTING_HOLE_4-40
- P1: footprint modular_device_teensy_3x2:DCJACK_2PIN_HIGHCURRENT_SMD_RA -> modular_device_base_3x2:DCJACK_2PIN_HIGHCURRENT_SMD_RA
- P2, P3, P4: footprint modular_device_teensy_3x2:Header_3_Pin_SMD_RA -> modular_device_base_3x2:Header_3_Pin_SMD_RA
- P5: footprint modular_device_teensy_3x2:BNC_DOUBLE -> modular_device_base_3x2:BNC_DOUBLE
- P6, P7: footprint modular_device_teensy_3x2:Header_2_Pin_SMD_RA -> modular_device_base_3x2:Header_2_Pin_SMD_RA
- REG1: footprint modular_device_teensy_3x2:DC_DC_CONV_R78C -> modular_device_base_3x2:DC_DC_CONV_R78C
- SW1: footprint modular_device_teensy_3x2:KT_SWITCH -> modular_device_base_3x2:KT_SWITCH
- TEENSY1: footprint modular_device_teensy_3x2:TEENSY_3 -> modular_device_base_3x2:TEENSY_3
Other:
- board text added: "Janelia Modular Device modular_device_base part_number: 1001 02/2017 ver 1.2 3x2"
- board text removed: "Janelia Modular Device modular_device_teensy part_number: 1001 02/2017 ver 1.2 3x2"
Changed lines of the file:
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@@
   (page A4)
   (title_block
-    (title modular_device_teensy_3x2)
+    (title modular_device_base_3x2)
     (rev 1.2)
   )
@@
     (add_net /TX3)
   )
-  (module modular_device_teensy_3x2:DO-214BA (layer B.Cu)
+  (module modular_device_base_3x2:DO-214BA (layer B.Cu)
     (at 71.755 113.665 270)
     (descr "Microsemi LSM115J")
@@
       (net 7 +5V))
   )
-  (module modular_device_teensy_3x2:SM1210 (layer B.Cu)
+  (module modular_device_base_3x2:SM1210 (layer B.Cu)
     (at 68.58 106.68)
     (tags "CMS SM")
@@
     )
   )
-  (module modular_device_teensy_3x2:SM1210 (layer B.Cu)
+  (module modular_device_base_3x2:SM1210 (layer B.Cu)
     (at 62.865 110.49 90)
     (tags "CMS SM")
@@
     )
   )
-  (module modular_device_teensy_3x2:Header_3_Pin_SMD_RA (layer B.Cu)
+  (module modular_device_base_3x2:Header_3_Pin_SMD_RA (layer B.Cu)
     (at 127.635 83.185 180)
     (fp_text reference P2 (at -5.715 -6.985 180) (layer B.SilkS)
@@
       (solder_mask_margin 0.1016) (clearance 0.1016))
   )
-  (module modular_device_teensy_3x2:Header_3_Pin_SMD_RA (layer F.Cu)
+  (module modular_device_base_3x2:Header_3_Pin_SMD_RA (layer F.Cu)
     (at 136.525 99.695 270)
     (fp_text reference P3 (at -5.715 6.985 270) (layer F.SilkS)
@@
       (solder_mask_margin 0.1016) (clearance 0.1016))
   )
-  (module modular_device_teensy_3x2:Header_3_Pin_SMD_RA (layer B.Cu)
+  (module modular_device_base_3x2:Header_3_Pin_SMD_RA (layer B.Cu)
     (at 127.635 116.205)
     (fp_text reference P4 (at -5.715 -6.985) (layer B.SilkS)
@@
       (solder_mask_margin 0.1016) (clearance 0.1016))
   )
-  (module modular_device_teensy_3x2:DC_DC_CONV_R78C (layer F.Cu)
+  (module modular_device_base_3x2:DC_DC_CONV_R78C (layer F.Cu)
     (at 67.31 113.03 270)
     (fp_text reference REG1 (at -0.635 -7.62 270) (layer F.SilkS)
@@
       (net 10 VDD))
   )
-  (module modular_device_teensy_3x2:BNC_DOUBLE (layer F.Cu)
+  (module modular_device_base_3x2:BNC_DOUBLE (layer F.Cu)
     (at 63.5 99.695 90)
     (fp_text reference P5 (at 0 11.43 90) (layer F.SilkS)
@@
       (net 2 GND))
   )
-  (module modular_device_teensy_3x2:KT_SWITCH (layer F.Cu)
+  (module modular_device_base_3x2:KT_SWITCH (layer F.Cu)
     (at 69.85 85.725 90)
     (fp_text reference SW1 (at 0 4.445 90) (layer F.SilkS)
@@
       (net 2 GND))
   )
-  (module modular_device_teensy_3x2:Header_2_Pin_SMD_RA (layer F.Cu)
+  (module modular_device_base_3x2:Header_2_Pin_SMD_RA (layer F.Cu)
     (at 127.635 81.915)
     (fp_text reference P6 (at -5.08 6.985 180) (layer F.SilkS)
@@
       (solder_mask_margin 0.1016) (clearance 0.1016))
   )
-  (module modular_device_teensy_3x2:Header_2_Pin_SMD_RA (layer F.Cu)
+  (module modular_device_base_3x2:Header_2_Pin_SMD_RA (layer F.Cu)
     (at 127.635 117.475 180)
     (fp_text reference P7 (at 5.08 6.985) (layer F.SilkS)
@@
       (solder_mask_margin 0.1016) (clearance 0.1016))
   )
-  (module modular_device_teensy_3x2:CFP15 (layer F.Cu)
+  (module modular_device_base_3x2:CFP15 (layer F.Cu)
     (at 118.11 109.22)
     (fp_text reference D4 (at -3.175 0 90) (layer F.SilkS)
@@
       (net 8 VCC) (solder_mask_margin 0.1) (clearance 0.1))
   )
-  (module modular_device_teensy_3x2:CFP15 (layer B.Cu)
+  (module modular_device_base_3x2:CFP15 (layer B.Cu)
     (at 64.135 99.695 90)
     (fp_text reference D3 (at 3.175 3.175 180) (layer B.SilkS)
@@
       (net 1 VAA) (solder_mask_margin 0.1) (clearance 0.1))
   )
-  (module modular_device_teensy_3x2:TEENSY_3 (layer B.Cu)
+  (module modular_device_base_3x2:TEENSY_3 (layer B.Cu)
     (at 95.25 99.695 270)
     (fp_text reference TEENSY1 (at 0 20.32 270) (layer B.SilkS)
@@
       (net 40 /D29))
   )
-  (module modular_device_teensy_3x2:SM1210 (layer B.Cu)
+  (module modular_device_base_3x2:SM1210 (layer B.Cu)
     (at 69.85 85.725 270)
     (tags "CMS SM")
@@
     )
   )
-  (module modular_device_teensy_3x2:SM1210 (layer B.Cu)
+  (module modular_device_base_3x2:SM1210 (layer B.Cu)
     (at 74.295 106.68 180)
     (tags "CMS SM")
@@
     )
   )
-  (module modular_device_teensy_3x2:SM1210 (layer F.Cu)
+  (module modular_device_base_3x2:SM1210 (layer F.Cu)
     (at 88.265 99.695)
     (tags "CMS SM")
@@
     )
   )
-  (module modular_device_teensy_3x2:DCJACK_2PIN_HIGHCURRENT_SMD_RA (layer B.Cu)
+  (module modular_device_base_3x2:DCJACK_2PIN_HIGHCURRENT_SMD_RA (layer B.Cu)
     (at 138.43 99.695 180)
     (fp_text reference P1 (at -7 -5.5 180) (layer B.SilkS)
@@
     (pad "" thru_hole circle (at 1.45 0 180) (size 2.2 2.2) (drill 1.8) (layers *.Cu *.Mask B.SilkS))
   )
-  (module modular_device_teensy_3x2:DO-214BA (layer F.Cu)
+  (module modular_device_base_3x2:DO-214BA (layer F.Cu)
     (at 81.28 99.695)
     (descr "Microsemi LSM115J")
@@
       (net 11 VEE))
   )
-  (module modular_device_teensy_3x2:MOUNTING_HOLE_4-40 (layer F.Cu)
+  (module modular_device_base_3x2:MOUNTING_HOLE_4-40 (layer F.Cu)
     (at 62.23 81.915)
     (fp_text reference MH1 (at 0 -3.175) (layer F.SilkS) hide
@@
     (pad 1 thru_hole circle (at 0 0) (size 3.556 3.556) (drill 3.302) (layers *.Cu *.Mask F.SilkS))
   )
-  (module modular_device_teensy_3x2:MOUNTING_HOLE_4-40 (layer F.Cu)
+  (module modular_device_base_3x2:MOUNTING_HOLE_4-40 (layer F.Cu)
     (at 62.23 117.475)
     (fp_text reference MH2 (at 0 -3.175) (layer F.SilkS) hide
@@
     (pad 1 thru_hole circle (at 0 0) (size 3.556 3.556) (drill 3.302) (layers *.Cu *.Mask F.SilkS))
   )
-  (module modular_device_teensy_3x2:MOUNTING_HOLE_4-40 (layer F.Cu)
+  (module modular_device_base_3x2:MOUNTING_HOLE_4-40 (layer F.Cu)
     (at 118.11 99.695)
     (fp_text reference MH3 (at 0 -3.175) (layer F.SilkS) hide
@@
     (pad 1 thru_hole circle (at 0 0) (size 3.556 3.556) (drill 3.302) (layers *.Cu *.Mask F.SilkS))
   )
-  (module modular_device_teensy_3x2:MODULAR_DEVICE_TEENSY_3X2_FEMALE (layer F.Cu)
+  (module modular_device_base_3x2:MODULAR_DEVICE_BASE_3X2_FEMALE (layer F.Cu)
     (at 95.25 99.695)
     (fp_text reference MDT1 (at 0 0) (layer F.SilkS) hide
       (effects (font (size 1.016 1.016) (thickness 0.254)))
     )
-    (fp_text value MODULAR_DEVICE_TEENSY_3X2_FEMALE (at 0 2.54) (layer F.SilkS) hide
+    (fp_text value MODULAR_DEVICE_BASE_3X2_FEMALE (at 0 2.54) (layer F.SilkS) hide
       (effects (font (thickness 0.3048)))
     )
@@
     (effects (font (size 1.016 1.016) (thickness 0.254)))
   )
-  (gr_text "Janelia Modular Device\nmodular_device_teensy\npart_number: 1001 02/2017 ver 1.2 3x2" (at 95.25 111.76) (layer B.SilkS)
+  (gr_text "Janelia Modular Device\nmodular_device_base\npart_number: 1001 02/2017 ver 1.2 3x2" (at 95.25 111.76) (layer B.SilkS)
     (effects (font (size 1.016 1.016) (thickness 0.254)) (justify mirror))
   )
@@
     (effects (font (size 1.016 1.016) (thickness 0.254)))
   )
-  (gr_text "Janelia Modular Device\nmodular_device_teensy\npart_number: 1001 02/2017 ver 1.2 3x2" (at 95.25 111.76) (layer F.SilkS)
+  (gr_text "Janelia Modular Device\nmodular_device_base\npart_number: 1001 02/2017 ver 1.2 3x2" (at 95.25 111.76) (layer F.SilkS)
     (effects (font (size 1.016 1.016) (thickness 0.254)))
   )

Commit message: modular_device_base_3x2_v1.2.
Parts:
- removed MDT1: MODULAR_DEVICE_BASE_3X2_FEMALE, modular_device_base_3x2:MODULAR_DEVICE_BASE_3X2_FEMALE
- added MDB1: MODULAR_DEVICE_BASE_3x2_FEMALE, footprints:MODULAR_DEVICE_BASE_3X2_FEMALE, F.Cu at (95.2, 99.7)
- TEENSY1: footprint modular_device_base_3x2:TEENSY_3 -> footprints:TEENSY_3.2
Routing:
- net GND: track 196.3 -> 233.6 mm
- net VCC: track 55.5 -> 23.8 mm, vias 0 -> 2
- net /RX1: track 55.6 -> 64.5 mm
- net /D12: track 17.6 -> 10.2 mm
- net /RX3: track 39.0 -> 46.4 mm, vias 0 -> 2
- net VEE: track 27.8 -> 34.8 mm, vias 0 -> 1
- net /BNC_A: track 41.8 -> 36.2 mm
- net /D24: track 32.2 -> 27.7 mm
- net /D25: track 32.2 -> 27.7 mm
- net /BNC_B: track 34.7 -> 31.0 mm
- net VDD: track 109.6 -> 106.1 mm
- net /TX3: track 49.9 -> 46.9 mm, vias 1 -> 3
- net /AREF: track 47.7 -> 44.6 mm
- net /TX1: track 47.8 -> 46.3 mm
- net /D28: track 19.9 -> 21.1 mm
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Other:
- net class Power: trace_width 1.0668 -> 1.016

Commit message: footprints: -> modular_device_base_3x2:.
Parts:
- MDB1: footprint footprints:MODULAR_DEVICE_BASE_3X2_FEMALE -> modular_device_base_3x2:MODULAR_DEVICE_BASE_3X2_FEMALE
- TEENSY1: footprint footprints:TEENSY_3.2 -> modular_device_base_3x2:TEENSY_3.2
Changed lines of the file:
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@@
     (pad 1 thru_hole circle (at 0 0) (size 3.556 3.556) (drill 3.302) (layers *.Cu *.Mask F.SilkS))
   )
-  (module footprints:MODULAR_DEVICE_BASE_3X2_FEMALE (layer F.Cu)
+  (module modular_device_base_3x2:MODULAR_DEVICE_BASE_3X2_FEMALE (layer F.Cu)
     (at 95.25 99.695)
     (fp_text reference MDB1 (at 0 0) (layer F.SilkS) hide
@@
     (pad "" thru_hole circle (at 22.86 -17.78) (size 3.556 3.556) (drill 3.302) (layers *.Cu *.Mask F.SilkS))
   )
-  (module footprints:TEENSY_3.2 (layer B.Cu)
+  (module modular_device_base_3x2:TEENSY_3.2 (layer B.Cu)
     (at 95.25 99.695 270)
     (fp_text reference TEENSY1 (at 0 -19.05 270) (layer B.SilkS)

Commit message: TEENSY_3_2 -> TEENSY_3.2.
Parts:
- MDB1: footprint modular_device_base_3x2:MODULAR_DEVICE_BASE_3X2_FEMALE -> footprints:MODULAR_DEVICE_BASE_3X2_FEMALE
- TEENSY1: value TEENSY_3_2 -> TEENSY_3.2; footprint modular_device_base_3x2:TEENSY_3.2 -> footprints:TEENSY_3.2
Changed lines of the file:
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@@
     (pad 1 thru_hole circle (at 0 0) (size 3.556 3.556) (drill 3.302) (layers *.Cu *.Mask F.SilkS))
   )
-  (module modular_device_base_3x2:MODULAR_DEVICE_BASE_3X2_FEMALE (layer F.Cu)
+  (module footprints:MODULAR_DEVICE_BASE_3X2_FEMALE (layer F.Cu)
     (at 95.25 99.695)
     (fp_text reference MDB1 (at 0 0) (layer F.SilkS) hide
@@
     (pad "" thru_hole circle (at 22.86 -17.78) (size 3.556 3.556) (drill 3.302) (layers *.Cu *.Mask F.SilkS))
   )
-  (module modular_device_base_3x2:TEENSY_3.2 (layer B.Cu)
+  (module footprints:TEENSY_3.2 (layer B.Cu)
     (at 95.25 99.695 270)
     (fp_text reference TEENSY1 (at 0 -19.05 270) (layer B.SilkS)
       (effects (font (size 1.016 1.016) (thickness 0.254)) (justify mirror))
     )
-    (fp_text value TEENSY_3_2 (at 0 16.5 270) (layer B.SilkS)
+    (fp_text value TEENSY_3.2 (at 0 16.5 270) (layer B.SilkS)
       (effects (font (size 1.016 1.016) (thickness 0.254)) (justify mirror))
     )

Commit message: Progress towards new modifications.
Parts:
- removed P7: HEADER_01X02_SMD_RA, modular_device_base_3x2:Header_2_Pin_SMD_RA
- added MH4: MNT_HOLE, modular_device_base_3x2:MOUNTING_HOLE_4-40, F.Cu at (118.1, 109.2)
- D3: moved to F.Cu
- P1: value PWR_JACK_2.5x5.5_SMD_RA -> PWR_JACK_2.5x5.5; footprint modular_device_base_3x2:DCJACK_2PIN_HIGHCURRENT_SMD_RA -> footprints:DCJACK_2PIN_HIGHCURRENT
- P2: value HEADER_01X03_SMD_RA -> BNC_DOUBLE_RA; footprint modular_device_base_3x2:Header_3_Pin_SMD_RA -> modular_device_base_3x2:BNC_DOUBLE; moved to F.Cu
- P3: moved to B.Cu
- P4: value HEADER_01X03_SMD_RA -> HEADER_01X02_SMD_RA; footprint modular_device_base_3x2:Header_3_Pin_SMD_RA -> modular_device_base_3x2:Header_2_Pin_SMD_RA; moved to F.Cu
- P5: value BNC_DOUBLE_RA -> HEADER_01X03_SMD_RA; footprint modular_device_base_3x2:BNC_DOUBLE -> modular_device_base_3x2:Header_3_Pin_SMD_RA; moved to B.Cu
- moved P5 66.8 mm to (128.3, 116.2), turned to 0 degrees
- moved P2 66.2 mm to (63.5, 99.7), turned to 90 degrees
- moved D3 61.6 mm to (125.7, 99.7), turned to 0 degrees
- moved P6 35.6 mm to (128.3, 117.5), turned to 180 degrees
- moved P4 34.3 mm to (128.3, 81.9)
- moved P3 18.5 mm to (128.3, 83.2), turned to 180 degrees
- moved D4 9.86 mm to (120.7, 99.7)
- moved MH3 9.52 mm to (118.1, 90.2)
- moved P1 5.08 mm to (143.5, 99.7), turned to 90 degrees
Connections:
- P2 pad 1: /RX1 -> /BNC_A
- P2 pad 3: /TX1 -> /BNC_B
- P3 pad 1: /RX2 -> /RX1
- P3 pad 3: /TX2 -> /TX1
- P4 pad 1: /RX3 -> VCC
- P5 pad 1: /BNC_A -> /RX3
- P5 pad 3: /BNC_B -> /TX3
- P6 pad 1: VCC -> GND
- P6 pad 2: GND -> VDD
- TEENSY1 pad 26: /RX2 -> (no net)
- TEENSY1 pad 31: /TX2 -> (no net)
Routing:
- net GND: track 233.6 -> 0.00 mm, vias 4 -> 0
- net VDD: track 106.1 -> 0.00 mm
- net VAA: track 89.5 -> 0.00 mm, vias 2 -> 0
- net /RX1: track 64.5 -> 0.00 mm, vias 1 -> 0
- net /PROG: track 58.2 -> 0.00 mm
- net /TX3: track 46.9 -> 0.00 mm, vias 3 -> 0
- net /RX3: track 46.4 -> 0.00 mm, vias 2 -> 0
- net /TX1: track 46.3 -> 0.00 mm, vias 1 -> 0
- net /AREF: track 44.6 -> 0.00 mm, vias 1 -> 0
- net /BNC_A: track 36.2 -> 0.00 mm
- net VEE: track 34.8 -> 0.00 mm, vias 1 -> 0
- net /BNC_B: track 31.0 -> 0.00 mm
- net /RX2: track 28.9 -> 0.00 mm
- net /TX2: track 28.8 -> 0.00 mm
- net /D25: track 27.7 -> 0.00 mm
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- removed copper zone on B.Cu, net GND
- removed copper zone on F.Cu, net GND
Other:
- board text removed: "Serial2"

Commit message: Finished design ver 1.0.
Parts:
- moved MH3 24.3 mm to (141.0, 81.9)
- moved MH4 24.3 mm to (141.0, 117.5)
- moved D4 4.49 mm to (123.8, 96.5), turned to 270 degrees
- moved D3 3.70 mm to (123.8, 102.9), turned to 270 degrees
- moved P3 0.64 mm to (127.6, 83.2)
- moved P4 0.64 mm to (127.6, 81.9)
- moved P5 0.64 mm to (127.6, 116.2)
- moved P6 0.64 mm to (127.6, 117.5)
Routing:
- net GND: track 0.00 -> 196.9 mm, vias 0 -> 1
- net VDD: track 0.00 -> 114.9 mm
- net /RX1: track 0.00 -> 58.0 mm
- net /PROG: track 0.00 -> 55.3 mm, vias 0 -> 1
- net /TX1: track 0.00 -> 48.6 mm
- net /D25: track 0.00 -> 44.5 mm
- net /BNC_A: track 0.00 -> 44.2 mm
- net /TX3: track 0.00 -> 41.9 mm
- net /RX3: track 0.00 -> 38.2 mm
- net VEE: track 0.00 -> 33.9 mm, vias 0 -> 1
- net /D24: track 0.00 -> 33.9 mm
- net /BNC_B: track 0.00 -> 31.0 mm
- net /AREF: track 0.00 -> 30.2 mm
- net /D30: track 0.00 -> 23.7 mm
- net /D29: track 0.00 -> 23.7 mm
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- added copper zone on B.Cu, net GND
- added copper zone on F.Cu, net VDD
Other:
- net class Power: trace_width 1.016 -> 1.2192
- board text added: "2.5x5.5 Center + +9-42VDC"
- board text added: "BNC A"
- board text added: "BNC B"
- board text added: "Janelia Modular Device modular_device_base part_number: 1001 02/2017 ver 1.0 3x2"
- board text removed: "+9-42VDC"
- board text removed: "2.5x5.5 Center +"
- board text removed: "Janelia Modular Device modular_device_base part_number: 1001 02/2017 ver 1.2 3x2"

Commit message: Progress towards v1.1.
Parts:
- added C6: 0.1uF, footprints:SM1210, B.Cu at (63.5, 99.7)
- added D5: diode_schottky_45V_10A, modular_device_base_3x2:CFP15, B.Cu at (119.4, 94.6)
- added D6: diode_schottky_45V_10A, modular_device_base_3x2:CFP15, F.Cu at (119.4, 97.2)
- added D7: diode_schottky_45V_10A, modular_device_base_3x2:CFP15, B.Cu at (119.4, 99.7)
- added D8: diode_schottky_45V_10A, modular_device_base_3x2:CFP15, F.Cu at (119.4, 107.3)
- added D9: diode_schottky_45V_10A, modular_device_base_3x2:CFP15, B.Cu at (119.4, 104.8)
- added L1: LED_5V_GRN_RA, footprints:LED_555-2XXX, F.Cu at (140.3, 108.0)
- added L2: LED_5V_YEL_RA, footprints:LED_555-2XXX, F.Cu at (140.3, 110.5)
- added U1: MAX6817, footprints:MAX6817, B.Cu at (69.2, 104.8)
- moved C3 54.5 mm to (118.1, 111.1), turned to 0 degrees
- moved SW1 27.9 mm to (69.8, 113.7)
- moved REG1 26.7 mm to (67.3, 86.4)
- moved C2 22.9 mm to (62.9, 87.6)
- moved C1 21.8 mm to (71.8, 85.1), turned to 270 degrees
- moved D2 21.0 mm to (71.1, 92.7), turned to 180 degrees
- moved D4 6.29 mm to (119.4, 92.1)
- moved D3 4.49 mm to (119.4, 102.2)
- moved C4 0.63 mm to (74.3, 107.3)
Connections:
- C1 pad 1: VDD -> VPP
- C3 pad 1: VDD -> VPP
- D3 pad 1: VDD -> VPP
- D4 pad 1: VDD -> VPP
- D4 pad 2: VCC -> VDD
- P6 pad 2: VDD -> VSS
- REG1 pad 1: VDD -> VPP
- SW1 pad 2: /PROG -> /BTN_A
- TEENSY1 pad 26: (no net) -> /LED_GRN
- TEENSY1 pad 27: (no net) -> /LED_YEL
- TEENSY1 pad 31: (no net) -> /BTN_A_D
- TEENSY1 pad PROG: /PROG -> (no net)
Routing:
- net GND: track 196.9 -> 0.00 mm, vias 1 -> 0
- net VDD: track 114.9 -> 0.00 mm
- net /RX1: track 58.0 -> 0.00 mm
- net /PROG: track 55.3 -> 0.00 mm, vias 1 -> 0
- net /TX1: track 48.6 -> 0.00 mm
- net /D25: track 44.5 -> 0.00 mm
- net /BNC_A: track 44.2 -> 0.00 mm
- net /TX3: track 41.9 -> 0.00 mm
- net /RX3: track 38.2 -> 0.00 mm
- net VEE: track 33.9 -> 0.00 mm, vias 1 -> 0
- net /D24: track 33.9 -> 0.00 mm
- net /BNC_B: track 31.0 -> 0.00 mm
- net /AREF: track 30.2 -> 0.00 mm
- net /D30: track 23.7 -> 0.00 mm
- net /D29: track 23.7 -> 0.00 mm
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- removed copper zone on B.Cu, net GND
- removed copper zone on F.Cu, net VDD
Other:
- board text added: "1"
- board text added: "3"
- board text added: "G"
- board text added: "GRN"
- board text added: "Janelia Modular Device modular_device_base part_number: 1001 05/2017 ver 1.1 3x2"
- board text added: "RX1"
- board text added: "RX3"
- board text added: "TX1"
- board text added: "TX3"
- board text added: "YEL"
- board text removed: "Janelia Modular Device modular_device_base part_number: 1001 02/2017 ver 1.0 3x2"
- board text removed: "Serial1"
- board text removed: "Serial3"

Commit message: Finished v1.1.
Parts:
- added L3: LED_5V_YEL_RA, footprints:LED_555-2XXX, F.Cu at (70.5, 116.8)
- added R1: 6.19k, footprints:SM1210, B.Cu at (118.1, 111.8)
- L1: value LED_5V_GRN_RA -> LED_5V_RED_RA; moved to B.Cu
- L2: value LED_5V_YEL_RA -> LED_5V_GRN_RA
- moved L2 72.7 mm to (67.9, 116.8), turned to 180 degrees
- moved C3 55.8 mm to (63.5, 99.7), turned to 270 degrees
- moved C6 11.4 mm to (63.5, 111.1), turned to 270 degrees
- moved U1 6.35 mm to (69.2, 111.1), turned to 180 degrees
- moved C4 4.02 mm to (70.5, 106.0)
- moved SW1 2.62 mm to (69.2, 111.1), turned to 0 degrees
- moved C2 0.90 mm to (63.5, 88.3)
- turned L1 to 90 degrees
Connections:
- L1 pad 1: /LED_GRN -> Net-(L1-Pad1)
- L2 pad 1: /LED_YEL -> /LED_GRN
Routing:
- net GND: track 0.00 -> 214.9 mm, vias 0 -> 1
- net VPP: track 0.00 -> 121.5 mm, vias 0 -> 2
- net /RX1: track 0.00 -> 83.8 mm, vias 0 -> 1
- net /LED_GRN: track 0.00 -> 83.2 mm, vias 0 -> 2
- net VEE: track 0.00 -> 74.3 mm, vias 0 -> 1
- net /LED_YEL: track 0.00 -> 71.2 mm
- net VDD: track 0.00 -> 61.1 mm, vias 0 -> 3
- net /TX3: track 0.00 -> 52.8 mm, vias 0 -> 2
- net /BTN_A_D: track 0.00 -> 51.9 mm, vias 0 -> 2
- net /TX1: track 0.00 -> 46.7 mm, vias 0 -> 1
- net /RX3: track 0.00 -> 42.1 mm, vias 0 -> 3
- net /BNC_A: track 0.00 -> 35.7 mm
- net /BNC_B: track 0.00 -> 34.1 mm
- net /D25: track 0.00 -> 28.8 mm
- net /D24: track 0.00 -> 28.5 mm
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- added copper zone on B.Cu, net GND
- added copper zone on F.Cu, net GND
Other:
- board text added: "R"
- board text added: "Top: BNC B Bot: BNC A"
- board text added: "Y"
- board text removed: "BNC A"
- board text removed: "BNC B"
- board text removed: "Bottom:"
- board text removed: "GRN"
- board text removed: "Top:"
- board text removed: "YEL"
