File: modular_device_base_3x2.kicad_pcb (KiCad board)
At the start: 2 copper layers, 85.1 x 41.9 mm, 35 parts, among them P1 PWR_JACK_2.5x5.5, P2 BNC_DOUBLE_RA, P3 HEADER_01X03_SMD_RA, P4 HEADER_01X02_SMD_RA, P5 HEADER_01X03_SMD_RA, P6 HEADER_01X02_SMD_RA, P7 HEADER_01X03_RA, SW1 KT_SWITCH, U1 MAX6817

Commit message: Progress towards v1.2.
Parts:
- added P8: HEADER_01X02_SMD_RA_UNSHR, footprints:Header_2_Pin_SMD_RA_UNSHR, B.Cu at (62.2, 111.1)
- moved C4 18.5 mm to (71.8, 87.6), turned to 90 degrees
- moved C6 9.67 mm to (72.4, 107.3), turned to 180 degrees
- moved U1 3.17 mm to (72.4, 111.1)
- moved C1 2.54 mm to (71.8, 82.5)
Connections:
- U1 pad 3: (no net) -> Net-(U1-Pad3)
- U1 pad 4: (no net) -> Net-(U1-Pad4)
Routing:
- net /RX1: track 61.0 -> 81.6 mm
- net /BTN_A_D: track 42.7 -> 62.5 mm, vias 1 -> 0
- net VEE: track 65.4 -> 49.6 mm, vias 0 -> 1
- net /BTN_A: track 4.04 -> 15.5 mm
- net /LED_GRN: track 51.8 -> 62.9 mm, vias 1 -> 0
- net Net-(P7-Pad2): track 34.3 -> 41.0 mm
- net /TX3: track 57.1 -> 50.6 mm, vias 0 -> 1
- net VPP: track 119.5 -> 126.0 mm, vias 2 -> 1
- net /AREF: track 26.7 -> 32.5 mm, vias 0 -> 2
- net /TX1: track 48.8 -> 43.6 mm, vias 2 -> 1
- net GND: track 256.2 -> 251.5 mm, vias 0 -> 1
- net /BNC_A: track 39.7 -> 35.7 mm
- net VSS: track 18.0 -> 15.4 mm
- net /D24: track 34.7 -> 32.2 mm, vias 0 -> 1
- net VDD: track 58.5 -> 60.8 mm, vias 2 -> 1
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- removed copper zone on B.Cu, net GND
- removed copper zone on F.Cu, net GND
Other:
- net class Default: clearance 0.2 -> 0
- rule trace_clearance: 0.2 -> 0
- board text added: "+12-42VDC"
- board text added: "2.5x5.5 Center + +12-42VDC"
- board text added: "DISABLE"
- board text added: "ENABLE"
- board text added: "Janelia Modular Device modular_device_base part_number: 1001 08/2017 ver 1.2 3x2"
- board text added: "RED LED"
- board text removed: "+9-42VDC"
- board text removed: "2.5x5.5 Center + +9-42VDC"
- board text removed: "Janelia Modular Device modular_device_base part_number: 1001 05/2017 ver 1.1 3x2"
- board text removed: "LED"
- board text removed: "OFF"
- board text removed: "ON"

Commit message: Finished v1.2.
Routing:
- added copper zone on B.Cu, net GND
- added copper zone on F.Cu, net GND
Changed lines of the file:
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@@
   (segment (start 118.3793 111.5395) (end 123.5637 111.5395) (width 0.6096) (layer B.Cu) (net 50))
   (segment (start 118.1588 111.76) (end 118.3793 111.5395) (width 0.6096) (layer B.Cu) (net 50))
+  (zone (net 2) (net_name GND) (layer F.Cu) (hatch edge 0.508)
+    (connect_pads (clearance 0.2032))
+    (min_thickness 0.2032)
+    (fill yes (arc_segments 16) (thermal_gap 0.508) (thermal_bridge_width 0.508))
+    (polygon
+      (pts
+        (xy 58.42 78.105) (xy 58.42 121.285) (xy 144.78 121.285) (xy 144.78 78.105)
+      )
+    )
+  )
+  (zone (net 2) (net_name GND) (layer B.Cu) (hatch edge 0.508)
+    (connect_pads (clearance 0.2032))
+    (min_thickness 0.2032)
+    (fill yes (arc_segments 16) (thermal_gap 0.508) (thermal_bridge_width 0.508))
+    (polygon
+      (pts
+        (xy 57.785 77.47) (xy 57.785 121.92) (xy 145.415 121.92) (xy 145.415 77.47)
+      )
+    )
+  )
 )
